Commit message: commit before removal of common

File: objects/cylinder.urdf (robot description, URDF)
Before this commit: robot simple cylinder, 1 links, 0 joints
Links:
- link my_cylinder: geometry collision box size=1 1 1; visual cylinder length=2 radius=0.2

Commit message: added record cylinder

File: objects/cylinder.urdf (robot description, URDF)
Before this commit: robot simple cylinder, 1 links, 0 joints
Links:
- link my_cylinder: mass 1.0 -> 1; geometry collision box size=0.6 0.6 0.6; visual cylinder length=2 radius=0.2

Commit message: pre merge goa-sf

File: objects/cylinder.urdf (robot description, URDF)
Before this commit: robot simple cylinder, 1 links, 0 joints
Links:
- link my_cylinder: geometry collision cylinder length=0.5 radius=0.2; visual cylinder length=0.5 radius=0.2

Commit message: pre-merge

File: objects/cylinder.urdf (robot description, URDF)
Before this commit: robot simple cylinder, 1 links, 0 joints
Links:
- link my_cylinder: geometry collision cylinder length=1.4 radius=0.2; visual cylinder length=1.4 radius=0.2
